Commit message: Symulacja w pelni sprawna

File: ros2_ws/src/robot_description/urdf/robot.urdf.xacro (robot description, xacro)
@@ -1,12 +1,36 @@
 <?xml version="1.0"?>
 <robot xmlns:xacro="http://www.ros.org/wiki/xacro" name="six_wheeled_robot">
+  <!-- ================= GEOMETRIA ================= -->
   <xacro:property name="base_length" value="0.2525"/>
   <xacro:property name="base_width"  value="0.126"/>
   <xacro:property name="base_height" value="0.094"/>
+  <xacro:property name="base_mass"   value="2.0"/> <!-- Dodana masa kadłuba [kg] -->
   <xacro:property name="wheel_radius" value="0.042"/>
   <xacro:property name="wheel_width"  value="0.0502"/>
+  <xacro:property name="wheel_mass"   value="0.2"/> <!-- Dodana masa koła [kg] -->
   <xacro:property name="wheel_x_offset" value="0.084"/>
   <xacro:property name="wheel_y_offset" value="${(base_width/2) + (wheel_width/2)}"/>
   <xacro:property name="wheel_z_offset" value="${-base_height/2}"/>
+  <!-- ================= MAKRA INERCJI ================= -->
+  <xacro:macro name="box_inertia" params="m w h d">
+    <inertial>
+      <origin xyz="0 0 0" rpy="0 0 0"/>
+      <mass value="${m}"/>
+      <!-- Zwróć uwagę na poprawione przypisanie zmiennych w w(width), h(height), d(depth/length) -->
+      <inertia ixx="${(m/12) * (w*w + h*h)}" ixy="0.0" ixz="0.0"
+               iyy="${(m/12) * (d*d + h*h)}" iyz="0.0"
+               izz="${(m/12) * (d*d + w*w)}"/>
+    </inertial>
+  </xacro:macro>
+  <xacro:macro name="cylinder_inertia" params="m r h">
+    <inertial>
+      <origin xyz="0 0 0" rpy="1.57079632679 0 0"/>
+      <mass value="${m}"/>
+      <inertia ixx="${(m/12) * (3*r*r + h*h)}" ixy="0" ixz="0"
+               iyy="${(m/12) * (3*r*r + h*h)}" iyz="0"
+               izz="${(m/2) * (r*r)}"/>
+    </inertial>
+  </xacro:macro>
+  <!-- ================= MATERIAŁY RVIZ ================= -->
   <material name="blue">
     <color rgba="0.0 0.0 0.8 1.0"/>
@@ -15,4 +39,13 @@
     <color rgba="0.1 0.1 0.1 1.0"/>
   </material>
+  <!-- ================= WIRTUALNY KORZEŃ (DLA SLAM I KDL) ================= -->
+  <link name="base_footprint"/>
+  <joint name="base_footprint_joint" type="fixed">
+    <parent link="base_footprint"/>
+    <child link="base_link"/>
+    <!-- Przesuwamy base_link w górę tak, by base_footprint "ślizgał się" idealnie po podłodze (Z=0) -->
+    <origin xyz="0 0 ${wheel_radius}" rpy="0 0 0"/>
+  </joint>
+  <!-- ================= KADŁUB ================= -->
   <link name="base_link">
     <visual>
@@ -27,5 +60,11 @@
       </geometry>
     </collision>
+    <!-- Fizyka kadłuba -->
+    <xacro:box_inertia m="${base_mass}" w="${base_width}" d="${base_length}" h="${base_height}"/>
   </link>
+  <gazebo reference="base_link">
+    <material>Gazebo/Blue</material>
+  </gazebo>
+  <!-- ================= MAKRO KOŁA ================= -->
   <xacro:macro name="wheel" params="name x y">
     <link name="${name}_link">
@@ -43,4 +82,6 @@
         </geometry>
       </collision>
+      <!-- Fizyka koła -->
+      <xacro:cylinder_inertia m="${wheel_mass}" r="${wheel_radius}" h="${wheel_width}"/>
     </link>
     <joint name="${name}_joint" type="continuous">
@@ -50,5 +91,11 @@
       <axis xyz="0 1 0"/>
     </joint>
+    <gazebo reference="${name}_link">
+      <material>Gazebo/Black</material>
+      <mu1>1.0</mu1>
+      <mu2>0.1</mu2>
+    </gazebo>
   </xacro:macro>
+  <!-- ================= INSTANCJE KÓŁ ================= -->
   <xacro:wheel name="front_left" x="${wheel_x_offset}"  y="${wheel_y_offset}"/>
   <xacro:wheel name="mid_left"   x="0.0"                y="${wheel_y_offset}"/>
@@ -57,3 +104,90 @@
   <xacro:wheel name="mid_right"   x="0.0"                y="-${wheel_y_offset}"/>
   <xacro:wheel name="rear_right"  x="-${wheel_x_offset}" y="-${wheel_y_offset}"/>
+  <!-- ================= WTYCZKA GAZEBO (NAPĘD 6x6) ================= -->
+  <gazebo>
+    <plugin name="diff_drive" filename="libgazebo_ros_diff_drive.so">
+      <update_rate>30.0</update_rate>
+      <!-- Parametr kluczowy dla 6 kół -->
+      <num_wheel_pairs>3</num_wheel_pairs>
+      <!-- Lewa strona -->
+      <left_joint>front_left_joint</left_joint>
+      <left_joint>mid_left_joint</left_joint>
+      <left_joint>rear_left_joint</left_joint>
+      <!-- Prawa strona -->
+      <right_joint>front_right_joint</right_joint>
+      <right_joint>mid_right_joint</right_joint>
+      <right_joint>rear_right_joint</right_joint>
+      <!-- Kinematyka wyliczona z parametrów XACRO -->
+      <wheel_separation>${2 * wheel_y_offset}</wheel_separation>
+      <wheel_diameter>${2 * wheel_radius}</wheel_diameter>
+      <!-- Ograniczenia -->
+      <max_wheel_torque>20</max_wheel_torque>
+      <max_wheel_acceleration>1.0</max_wheel_acceleration>
+      <!-- Wyjścia (Odometria i TF) -->
+      <publish_odom>true</publish_odom>
+      <publish_odom_tf>true</publish_odom_tf>
+      <publish_wheel_tf>true</publish_wheel_tf>
+      <odometry_frame>odom</odometry_frame>
+      <robot_base_frame>base_footprint</robot_base_frame>
+    </plugin>
+  </gazebo>
+  <!--LIDAR-->
+  <xacro:property name="lidar_radius" value="0.035"/>
+  <xacro:property name="lidar_height" value="0.055"/>
+  <xacro:property name="lidar_mass"   value="0.190"/>
+  <link name="lidar_link">
+    <visual>
+      <geometry>
+        <cylinder radius="${lidar_radius}" length="${lidar_height}"/>
+      </geometry>
+      <material name="black"/>
+    </visual>
+    <collision>
+      <geometry>
+        <cylinder radius="${lidar_radius}" length="${lidar_height}"/>
+      </geometry>
+    </collision>
+    <inertial>
+      <origin xyz="0 0 0" rpy="0 0 0"/>
+      <mass value="${lidar_mass}"/>
+      <inertia ixx="${(lidar_mass/12) * (3*lidar_radius*lidar_radius + lidar_height*lidar_height)}" ixy="0" ixz="0"
+               iyy="${(lidar_mass/12) * (3*lidar_radius*lidar_radius + lidar_height*lidar_height)}" iyz="0"
+               izz="${(lidar_mass/2) * (lidar_radius*lidar_radius)}"/>
+    </inertial>
+  </link>
+  <joint name="lidar_joint" type="fixed">
+    <parent link="base_link"/>
+    <child link="lidar_link"/>
+    <origin xyz="0 0 ${base_height/2 + lidar_height/2}" rpy="0 0 0"/>
+  </joint>
+  <gazebo reference="lidar_link">
+    <material>Gazebo/Black</material>
+    <sensor type="ray" name="rplidar_a1_sensor">
+      <pose>0 0 0 0 0 0</pose>
+      <visualize>true</visualize>
+      <update_rate>5.5</update_rate>
+      <ray>
+        <scan>
+          <horizontal>
+            <samples>360</samples>
+            <resolution>1</resolution>
+            <min_angle>-3.14159</min_angle>
+            <max_angle>3.14159</max_angle>
+          </horizontal>
+        </scan>
+        <range>
+          <min>0.15</min>
+          <max>12.0</max>
+          <resolution>0.01</resolution>
+        </range>
+      </ray>
+      <plugin name="gazebo_ros_lidar" filename="libgazebo_ros_ray_sensor.so">
+        <ros>
+          <argument>~/out:=scan</argument>
+        </ros>
+        <output_type>sensor_msgs/LaserScan</output_type>
+        <frame_name>lidar_link</frame_name>
+      </plugin>
+    </sensor>
+  </gazebo>
 </robot>

Commit message: Dodanie środowiska symulacyjnego (Gazebo + RViz2): kamera głębi OAK-D Lite, testowy świat z przeszkodami, konfiguracja RViz. Dokumentacja w docs/SIMULATION_CHANGES.md

File: ros2_ws/src/robot_description/urdf/robot.urdf.xacro (robot description, xacro)
@@ -191,3 +191,65 @@
     </sensor>
   </gazebo>
+  <!--KAMERA GŁĘBI OAK-D LITE-->
+  <xacro:property name="cam_length" value="0.091"/>
+  <xacro:property name="cam_width"  value="0.028"/>
+  <xacro:property name="cam_height" value="0.018"/>
+  <xacro:property name="cam_mass"   value="0.061"/>
+  <link name="camera_link">
+    <visual>
+      <geometry>
+        <box size="${cam_length} ${cam_width} ${cam_height}"/>
+      </geometry>
+      <material name="black"/>
+    </visual>
+    <collision>
+      <geometry>
+        <box size="${cam_length} ${cam_width} ${cam_height}"/>
+      </geometry>
+    </collision>
+    <xacro:box_inertia m="${cam_mass}" w="${cam_width}" d="${cam_length}" h="${cam_height}"/>
+  </link>
+  <joint name="camera_joint" type="fixed">
+    <parent link="base_link"/>
+    <child link="camera_link"/>
+    <!-- montaż na przedniej krawędzi kadłuba, u góry -->
+    <origin xyz="${base_length/2} 0 ${base_height/2}" rpy="0 0 0"/>
+  </joint>
+  <!-- Ramka "optyczna" (konwencja ROS- Z do przodu) - wymagana żeby obraz/chmura punktów miały poprawną orientację -->
+  <link name="camera_link_optical"/>
+  <joint name="camera_optical_joint" type="fixed">
+    <parent link="camera_link"/>
+    <child link="camera_link_optical"/>
+    <origin xyz="0 0 0" rpy="-1.57079632679 0 -1.57079632679"/>
+  </joint>
+  <gazebo reference="camera_link">
+    <material>Gazebo/Black</material>
+    <sensor type="depth" name="oak_d_lite_depth">
+      <update_rate>15</update_rate>
+      <camera>
+        <horizontal_fov>1.204</horizontal_fov> <!-- ~69 st. FOV RGB, OAK-D Lite -->
+        <image>
+          <width>640</width>
+          <height>480</height>
+          <format>B8G8R8</format>
+        </image>
+        <clip>
+          <near>0.1</near>
+          <far>10.0</far>
+        </clip>
+      </camera>
+      <plugin name="oak_d_lite_controller" filename="libgazebo_ros_camera.so">
+        <ros>
+          <namespace>sniff</namespace>
+          <remapping>image_raw:=camera/color/image_raw</remapping>
+          <remapping>camera_info:=camera/color/camera_info</remapping>
+          <remapping>depth/image_raw:=camera/depth/image_raw</remapping>
+          <remapping>points:=camera/depth/points</remapping>
+        </ros>
+        <frame_name>camera_link_optical</frame_name>
+        <min_depth>0.1</min_depth> # zmienić na 0.2 - w domyśle metry
+        <max_depth>50.0</max_depth> #zmienić na 12.0 bo takie są ograniczenia OAK-D lite kamery
+      </plugin>
+    </sensor>
+  </gazebo>
 </robot>

Commit message: naprawa pliku urdf

File: ros2_ws/src/robot_description/urdf/robot.urdf.xacro (robot description, xacro)
@@ -41,9 +41,8 @@
   <!-- ================= WIRTUALNY KORZEŃ (DLA SLAM I KDL) ================= -->
   <link name="base_footprint"/>
-  <joint name="base_footprint_joint" type="fixed">
+    <joint name="base_footprint_joint" type="fixed">
     <parent link="base_footprint"/>
     <child link="base_link"/>
-    <!-- Przesuwamy base_link w górę tak, by base_footprint "ślizgał się" idealnie po podłodze (Z=0) -->
-    <origin xyz="0 0 ${wheel_radius}" rpy="0 0 0"/>
+    <origin xyz="0 0 ${wheel_radius - wheel_z_offset}" rpy="0 0 0"/>
   </joint>
   <!-- ================= KADŁUB ================= -->
@@ -108,5 +107,4 @@
     <plugin name="diff_drive" filename="libgazebo_ros_diff_drive.so">
       <update_rate>30.0</update_rate>
-      <!-- Parametr kluczowy dla 6 kół -->
       <num_wheel_pairs>3</num_wheel_pairs>
       <!-- Lewa strona -->
@@ -118,14 +116,16 @@
       <right_joint>mid_right_joint</right_joint>
       <right_joint>rear_right_joint</right_joint>
-      <!-- Kinematyka wyliczona z parametrów XACRO -->
+      <!-- KLUCZOWE: po jednym wpisie NA KAŻDĄ PARĘ -->
+      <wheel_separation>${2 * wheel_y_offset}</wheel_separation>
+      <wheel_separation>${2 * wheel_y_offset}</wheel_separation>
       <wheel_separation>${2 * wheel_y_offset}</wheel_separation>
       <wheel_diameter>${2 * wheel_radius}</wheel_diameter>
-      <!-- Ograniczenia -->
+      <wheel_diameter>${2 * wheel_radius}</wheel_diameter>
+      <wheel_diameter>${2 * wheel_radius}</wheel_diameter>
       <max_wheel_torque>20</max_wheel_torque>
       <max_wheel_acceleration>1.0</max_wheel_acceleration>
-      <!-- Wyjścia (Odometria i TF) -->
       <publish_odom>true</publish_odom>
       <publish_odom_tf>true</publish_odom_tf>
-      <publish_wheel_tf>true</publish_wheel_tf>
+      <publish_wheel_tf>false</publish_wheel_tf>
       <odometry_frame>odom</odometry_frame>
       <robot_base_frame>base_footprint</robot_base_frame>

Commit message: poprawka modelu

File: ros2_ws/src/robot_description/urdf/robot.urdf.xacro (robot description, xacro)
@@ -132,4 +132,36 @@
     </plugin>
   </gazebo>
+<!-- ================= OBUDOWA (WIEZA POD LIDAR) ================= -->
+  <xacro:property name="tower_height" value="0.36"/>
+  <xacro:property name="tower_size_x" value="0.289"/>
+  <xacro:property name="tower_size_y" value="0.23"/>
+  <xacro:property name="tower_mass"   value="0.15"/>
+  <!-- Origin modelu STL lezy w globalnym ukladzie CAD (X~636, Y~918, Z~1270 mm).
+       Przesuwamy go tak, zeby srodek podstawy wypadl w (0,0,0). -->
+  <link name="tower_link">
+    <visual>
+      <origin xyz="-0.751 1.385 -0.918" rpy="1.5708 0 0"/>
+      <geometry>
+        <mesh filename="package://robot_description/meshes/obudowa.stl"
+              scale="0.001 0.001 0.001"/>
+      </geometry>
+      <material name="black"/>
+    </visual>
+    <collision>
+      <origin xyz="0 0 ${tower_height/2}" rpy="0 0 0"/>
+      <geometry>
+        <box size="${tower_size_x} ${tower_size_y} ${tower_height}"/>
+      </geometry>
+    </collision>
+    <xacro:box_inertia m="${tower_mass}" w="${tower_size_y}" d="${tower_size_x}" h="${tower_height}"/>
+  </link>
+  <joint name="tower_joint" type="fixed">
+    <parent link="base_link"/>
+    <child link="tower_link"/>
+    <origin xyz="0 0 ${base_height/2}" rpy="0 0 0"/>
+  </joint>
+  <gazebo reference="tower_link">
+    <material>Gazebo/Black</material>
+  </gazebo>
   <!--LIDAR-->
   <xacro:property name="lidar_radius" value="0.035"/>
@@ -157,7 +189,7 @@
   </link>
   <joint name="lidar_joint" type="fixed">
-    <parent link="base_link"/>
+    <parent link="tower_link"/>
     <child link="lidar_link"/>
-    <origin xyz="0 0 ${base_height/2 + lidar_height/2}" rpy="0 0 0"/>
+    <origin xyz="0 0 ${tower_height + lidar_height/2}" rpy="0 0 0"/>
   </joint>
   <gazebo reference="lidar_link">
